Commit message: Fix everything

File: car_description/urdf/base_link.xacro (robot description, xacro)
@@ -136,3 +136,28 @@
         </plugin>
     </gazebo>
+    <ros2_control name="f1tenth_mock_hw" type="system">
+      <hardware>
+        <plugin>mock_components/GenericSystem</plugin>
+      </hardware>
+      <joint name="right_rear_wheel_joint">
+        <command_interface name="velocity"/>
+        <state_interface name="position"/>
+        <state_interface name="velocity"/>
+      </joint>
+      <joint name="left_rear_wheel_joint">
+        <command_interface name="velocity"/>
+        <state_interface name="velocity"/>
+        <state_interface name="position"/>
+      </joint>
+      <joint name="right_steering_hinge_joint">
+        <command_interface name="position"/>
+        <state_interface name="velocity"/>
+        <state_interface name="position"/>
+      </joint>
+      <joint name="left_steering_hinge_joint">
+        <command_interface name="position"/>
+        <state_interface name="velocity"/>
+        <state_interface name="position"/>
+      </joint>
+    </ros2_control>
 </robot>
